Commit message: init

File: src/a600_description/xacro/a600_description.xacro (robot description, xacro)
@@ -8,5 +8,5 @@
 <xacro:property name="lower_angle" value="-1.04719755"/>
 <xacro:property name="upper_angle" value="1.04719755"/>
-<xacro:property name="effort" value="1000"/>
+<xacro:property name="effort" value="10000"/>
 <xacro:property name="angular_velocity" value="0.5"/>
 <!-- <link name="dummy">

File: src/a600_description/xacro/links_joints.xacro (robot description, xacro)
@@ -61,8 +61,8 @@
       <type>transmission_interface/SimpleTransmission</type>
       <joint name="${name}">
-        <hardwareInterface>hardware_interface/PositionJointInterface</hardwareInterface>
+        <hardwareInterface>hardware_interface/EffortJointInterface</hardwareInterface>
       </joint>
       <actuator name="motor_${name}">
-        <hardwareInterface>hardware_interface/PositionJointInterface</hardwareInterface>
+        <hardwareInterface>hardware_interface/EffortJointInterface</hardwareInterface>
         <mechanicalReduction>1</mechanicalReduction>
       </actuator>

Commit message: light mesh

File: src/a600_description/xacro/a600_description.xacro (robot description, xacro)
@@ -8,6 +8,11 @@
 <xacro:property name="lower_angle" value="-1.04719755"/>
 <xacro:property name="upper_angle" value="1.04719755"/>
-<xacro:property name="effort" value="10000"/>
 <xacro:property name="angular_velocity" value="0.5"/>
+<xacro:property name="HipR_max_effort" value="60"/>
+<xacro:property name="HipS_max_effort" value="250"/>
+<xacro:property name="HipF_max_effort" value="220"/>
+<xacro:property name="Knee_max_effort" value="220"/>
+<xacro:property name="FootF_max_effort" value="220"/>
+<xacro:property name="FootS_max_effort" value="10000"/>
 <!-- <link name="dummy">
    </link>
@@ -40,5 +45,5 @@
         origin_rpy="1.5708 0 0" origin_xyz="-0.088 -0.027645 0"
         parent="base_link" child="R_HipR"
-        limit_e="${effort}" limit_l="${lower_angle}" limit_u="${upper_angle}" limit_v="${angular_velocity}"
+        limit_e="${HipR_max_effort}" limit_l="${lower_angle}" limit_u="${upper_angle}" limit_v="${angular_velocity}"
         axis_xyz="0 1 0" />
 <link_stl name="R_HipS"
@@ -57,5 +62,5 @@
         origin_rpy="3.1416 0 3.1416"
         parent="R_HipR" child="R_HipS"
-        limit_e="${effort}" limit_l="${lower_angle}" limit_u="${upper_angle}" limit_v="${angular_velocity}"
+        limit_e="${HipS_max_effort}" limit_l="${lower_angle}" limit_u="${upper_angle}" limit_v="${angular_velocity}"
         axis_xyz="0 0 1" />
 <link_stl name="R_Knee_Upper"
@@ -70,9 +75,9 @@
         izz="0.039371"
         color = 'orange' />
-<revolute_joint name="R_Knee_Upper" type="revolute"
+<revolute_joint name="R_HipF" type="revolute"
       origin_xyz="0 0 0"
       origin_rpy="0 0 0"
         parent="R_HipS" child="R_Knee_Upper"
-        limit_e="${effort}" limit_l="${lower_angle}" limit_u="${upper_angle}" limit_v="${angular_velocity}"
+        limit_e="${HipF_max_effort}" limit_l="${lower_angle}" limit_u="${upper_angle}" limit_v="${angular_velocity}"
         axis_xyz="1 0 0" />
 <link_stl name="R_Knee_Lower"
@@ -87,9 +92,9 @@
         izz="0.015199"
         color = 'orange' />
-<revolute_joint name="R_Knee_Lower" type="revolute"
+<revolute_joint name="R_Knee" type="revolute"
       origin_xyz="0 -0.28 0"
       origin_rpy="3.1416 0 3.1416"
         parent="R_Knee_Upper" child="R_Knee_Lower"
-        limit_e="${effort}" limit_l="${lower_angle}" limit_u="${upper_angle}" limit_v="${angular_velocity}"
+        limit_e="${Knee_max_effort}" limit_l="${lower_angle}" limit_u="${upper_angle}" limit_v="${angular_velocity}"
         axis_xyz="1 0 0" />
 <link_stl name="R_FootR"
@@ -104,9 +109,9 @@
         izz="0.0003019"
         color = 'orange' />
-<revolute_joint name="R_FootR" type="revolute"
+<revolute_joint name="R_FootF" type="revolute"
       origin_xyz="0 -0.27682 0.010063"
       origin_rpy="3.1053 -0.00039391 -0.010836"
         parent="R_Knee_Lower" child="R_FootR"
-        limit_e="${effort}" limit_l="${lower_angle}" limit_u="${upper_angle}" limit_v="${angular_velocity}"
+        limit_e="${FootF_max_effort}" limit_l="${lower_angle}" limit_u="${upper_angle}" limit_v="${angular_velocity}"
         axis_xyz="0.99994 -0.010843 0"   />
 <link_stl name="R_FootS"
@@ -125,5 +130,5 @@
       origin_rpy="0 0 0"
         parent="R_FootR" child="R_FootS"
-        limit_e="${effort}" limit_l="${lower_angle}" limit_u="${upper_angle}" limit_v="${angular_velocity}"
+        limit_e="${FootS_max_effort}" limit_l="${lower_angle}" limit_u="${upper_angle}" limit_v="${angular_velocity}"
         axis_xyz="0 0 1"  />
 <!-- Left Leg -->
@@ -143,5 +148,5 @@
       origin_rpy="1.5708 0 0"
         parent="base_link" child="L_HipR"
-        limit_e="${effort}" limit_l="${lower_angle}" limit_u="${upper_angle}" limit_v="${angular_velocity}"
+        limit_e="${HipR_max_effort}" limit_l="${lower_angle}" limit_u="${upper_angle}" limit_v="${angular_velocity}"
         axis_xyz="0 1 0"  />
 <link_stl name="L_HipS"
@@ -160,5 +165,5 @@
       origin_rpy="0 0 0"
         parent="L_HipR" child="L_HipS"
-        limit_e="${effort}" limit_l="${lower_angle}" limit_u="${upper_angle}" limit_v="${angular_velocity}"
+        limit_e="${HipS_max_effort}" limit_l="${lower_angle}" limit_u="${upper_angle}" limit_v="${angular_velocity}"
         axis_xyz="0 0 1"  />
 <link_stl name="L_Knee_upper"
@@ -173,9 +178,9 @@
         izz="0.039943"
         color = 'orange' />
-<revolute_joint name="L_Knee_upper" type="revolute"
+<revolute_joint name="L_HipF" type="revolute"
       origin_xyz="0 0 0"
       origin_rpy="0 0 0"
         parent="L_HipS" child="L_Knee_upper"
-        limit_e="${effort}" limit_l="${lower_angle}" limit_u="${upper_angle}" limit_v="${angular_velocity}"
+        limit_e="${HipF_max_effort}" limit_l="${lower_angle}" limit_u="${upper_angle}" limit_v="${angular_velocity}"
         axis_xyz="1 0 0"  />
 <link_stl name="L_Knee_Lower"
@@ -190,9 +195,9 @@
         izz="0.01553"
         color = 'orange' />
-<revolute_joint name="L_Knee_Lower" type="revolute"
+<revolute_joint name="L_Knee" type="revolute"
       origin_xyz="0 -0.28 0"
       origin_rpy="-0.036336 0 0"
         parent="L_Knee_upper" child="L_Knee_Lower"
-        limit_e="${effort}" limit_l="${lower_angle}" limit_u="${upper_angle}" limit_v="${angular_velocity}"
+        limit_e="${Knee_max_effort}" limit_l="${lower_angle}" limit_u="${upper_angle}" limit_v="${angular_velocity}"
         axis_xyz="1 0 0"  />
 <link_stl name="L_FootR"
@@ -207,9 +212,9 @@
         izz="0.0003019"
         color = 'orange' />
-<revolute_joint name="L_FootR" type="revolute"
+<revolute_joint name="L_FootF" type="revolute"
       origin_xyz="0 -0.277 0"
       origin_rpy="3.1416 0 -0.010843"
         parent="L_Knee_Lower" child="L_FootR"
-        limit_e="${effort}" limit_l="${lower_angle}" limit_u="${upper_angle}" limit_v="${angular_velocity}"
+        limit_e="${FootF_max_effort}" limit_l="${lower_angle}" limit_u="${upper_angle}" limit_v="${angular_velocity}"
         axis_xyz="0.99994 -0.010843 0"  />
 <link_stl name="L_FootS"
@@ -228,5 +233,5 @@
       origin_rpy="0 0 0"
         parent="L_FootR" child="L_FootS"
-        limit_e="${effort}" limit_l="${lower_angle}" limit_u="${upper_angle}" limit_v="${angular_velocity}"
+        limit_e="${FootS_max_effort}" limit_l="${lower_angle}" limit_u="${upper_angle}" limit_v="${angular_velocity}"
         axis_xyz="0 0 1"  />
 </robot>

File: src/a600_description/xacro/links_joints.xacro (robot description, xacro)
@@ -12,5 +12,5 @@
         <origin rpy="0 0 0" xyz="0 0 0" />
           <geometry>
-            <mesh filename="package://a600_description/meshes/${name}.STL" />
+            <mesh filename="package://a600_description/meshes_light/${name}.STL" />
           </geometry>
       </collision>
@@ -18,5 +18,5 @@
         <origin rpy="0 0 0" xyz="0 0 0" />
         <geometry>
-            <mesh filename="package://a600_description/meshes/${name}.STL" />
+            <mesh filename="package://a600_description/meshes_light/${name}.STL" />
         </geometry>
           <material name="${color}"/>
@@ -42,5 +42,5 @@
         <origin rpy="0 0 0" xyz="0 0 0" />
         <geometry>
-            <mesh filename="package://a600_description/meshes/${name}.STL" />
+            <mesh filename="package://a600_description/meshes_light/${name}.STL" />
         </geometry>
           <material name="${color}"/>
