Commit message: colisions are corrected

File: src/a600_description/xacro/a600_description_box_colision.xacro (robot description, xacro)
@@ -2,5 +2,6 @@
 <robot name="AR-600" xmlns:xacro="http://www.ros.org/wiki/xacro">
 <!-- Start - Include -->
-  <xacro:include filename="$(find a600_description)/xacro/links_joints.xacro"/>
+  <xacro:include filename="$(find a600_description)/xacro/links_joints_macro.xacro"/>
+  <xacro:include filename="$(find a600_description)/xacro/a600_links_description.xacro"/>
   <xacro:include filename="$(find a600_description)/xacro/plugin.gazebo"/>
   <!-- Constants value-->
@@ -8,241 +9,129 @@
 <xacro:property name="lower_angle" value="-1.04719755"/>
 <xacro:property name="upper_angle" value="1.04719755"/>
-<xacro:property name="angular_velocity" value="0.5"/>
-<xacro:property name="HipR_max_effort" value="60"/>
-<xacro:property name="HipS_max_effort" value="250"/>
-<xacro:property name="HipF_max_effort" value="220"/>
-<xacro:property name="Knee_max_effort" value="220"/>
-<xacro:property name="FootF_max_effort" value="220"/>
-<xacro:property name="FootS_max_effort" value="10000"/>
-<!-- <link name="dummy">
-   </link>
-  <joint name="dummy_joint" type="fixed">
-     <parent link="dummy"/>
-     <child link="body"/>
-   </joint> -->
-<link_stl_box name="base_link"
-        origin_xyz="-0.0014901 0.13851 0.00071357" origin_rpy="0 0 0"
-        box_size = "0.001 0.001 0.001"
-        mass="28.386"
-        ixx="0.073017"
-        ixy="-3.603E-05"
-        ixz="5.7649E-06"
-        iyy="0.085864"
-        iyz="0.0040898"
-        izz="0.10252"
-        color = 'orange' />
-<!-- Right Leg -->
-<link_stl_box name="R_HipR"
-        origin_xyz="0.00071161 -0.027458 -0.023065" origin_rpy="0 0 0"
-        box_size = "0.001 0.001 0.001"
-        mass="2.3558"
-        ixx="0.0032395"
-        ixy="1.8675E-05"
-        ixz="-4.6222E-05"
-        iyy="0.0032177"
-        iyz="7.5574E-06"
-        izz="0.0025538"
-        color = 'orange' />
+<!-- velocity value-->
+<xacro:property name="angular_velocity_hip" value="2.5"/>
+<xacro:property name="angular_velocity_knee" value="5.8"/>
+<xacro:property name="angular_velocity_foot" value="3.4"/>
+<!-- Efforts value-->
+<xacro:property name="HipR_max_effort" value="60.0"/>
+<xacro:property name="HipS_max_effort" value="250.0"/>
+<xacro:property name="HipF_max_effort" value="250.0"/>
+<xacro:property name="Knee_max_effort" value="220.0"/>
+<xacro:property name="FootF_max_effort" value="60.0"/>
+<xacro:property name="FootS_max_effort" value="60.0"/>
+<!-- Foot pid value-->
+<xacro:property name="ground_kp"  value="1000000.0" />
+<xacro:property name="ground_kd"  value="10000.0" />
+<xacro:property name="ground_mu1"  value="1.5" />
+<xacro:property name="ground_mu2"  value="1.5" />
+<!-- Friction damping value-->
+<xacro:property name="leg_joint_damping"  value="0.1" />
+<xacro:property name="leg_joint_friction"  value="10" />
+<!-- Joint decription-->
 <revolute_joint name="R_HipR" type="revolute"
-        origin_rpy="1.5708 0 0" origin_xyz="-0.088 -0.027645 0"
+        origin_rpy="1.5708 0 0"
+        origin_xyz="-0.088 -0.027645 0"
         parent="base_link" child="R_HipR"
-        limit_e="${HipR_max_effort}" limit_l="${lower_angle}" limit_u="${upper_angle}" limit_v="${angular_velocity}"
+        limit_e="${HipR_max_effort}" limit_l="-0.175" limit_u="0.175" limit_v="${angular_velocity_hip}"
+        joint_damping ="${leg_joint_damping}"  joint_friction ="${leg_joint_friction}"
         axis_xyz="0 1 0" />
-<link_stl_box name="R_HipS"
-        origin_xyz="0.0032793 0.00011106 0.025957"
-        origin_rpy="0 0 0"
-        box_size = "0.001 0.001 0.001"
-        mass="6.15"
-        ixx="0.0051093"
-        ixy="1.2709E-05"
-        ixz="7.1765E-06"
-        iyy="0.0048779"
-        iyz="-5.4798E-06"
-        izz="0.0062721"
-        color = 'orange' />
 <revolute_joint name="R_HipS" type="revolute"
         origin_xyz="0 -0.102 0"
         origin_rpy="3.1416 0 3.1416"
         parent="R_HipR" child="R_HipS"
-        limit_e="${HipS_max_effort}" limit_l="${lower_angle}" limit_u="${upper_angle}" limit_v="${angular_velocity}"
+        limit_e="${HipS_max_effort}" limit_l="-0.192" limit_u="0.314" limit_v="${angular_velocity_hip}"
+        joint_damping ="${leg_joint_damping}"  joint_friction ="${leg_joint_friction}"
         axis_xyz="0 0 1" />
-<link_stl_box name="R_Knee_Upper"
-        origin_xyz="0.018772 -0.22402 -0.0063916"
+<revolute_joint name="R_HipF" type="revolute"
+        origin_xyz="0 0 0"
         origin_rpy="0 0 0"
-        box_size = "0.001 0.001 0.001"
-        mass="16.331"
-        ixx="0.048034"
-        ixy="2.0407E-07"
-        ixz="-6.8084E-05"
-        iyy="0.015142"
-        iyz="-0.00213"
-        izz="0.039371"
-        color = 'orange' />
-<revolute_joint name="R_HipF" type="revolute"
-      origin_xyz="0 0 0"
-      origin_rpy="0 0 0"
         parent="R_HipS" child="R_Knee_Upper"
-        limit_e="${HipF_max_effort}" limit_l="${lower_angle}" limit_u="${upper_angle}" limit_v="${angular_velocity}"
+        limit_e="${HipF_max_effort}" limit_l="-1.047" limit_u="0.698" limit_v="${angular_velocity_hip}"
+        joint_damping ="${leg_joint_damping}"  joint_friction ="${leg_joint_friction}"
         axis_xyz="1 0 0" />
-<link_stl_box name="R_Knee_Lower"
-        origin_xyz="-0.011938 -0.17383 0.0029031"
+<revolute_joint name="R_Knee" type="revolute"
+        origin_xyz="0 -0.28 0"
+        origin_rpy="3.1416 0 3.1416"
+        parent="R_Knee_Upper" child="R_Knee_Lower"
+        limit_e="${Knee_max_effort}" limit_l="-0.087" limit_u="1.571" limit_v="${angular_velocity_knee}"
+        joint_damping ="${leg_joint_damping}"  joint_friction ="${leg_joint_friction}"
+        axis_xyz="1 0 0" />
+<revolute_joint name="R_FootF" type="revolute"
+        origin_xyz="0 -0.277 0.0"
+        origin_rpy="3.1416 0 0"
+        parent="R_Knee_Lower" child="R_FootR"
+        limit_e="${FootF_max_effort}" limit_l="-1.047" limit_u="0.559" limit_v="${angular_velocity_foot}"
+        joint_damping ="${leg_joint_damping}"  joint_friction ="${leg_joint_friction}"
+        axis_xyz="1 0 0"   />
+<revolute_joint name="R_FootS" type="revolute"
+        origin_xyz="0 0.030 0"
         origin_rpy="0 0 0"
-        box_size = "0.001 0.001 0.001"
-        mass="10.03"
-        ixx="0.020389"
-        ixy="3.5365E-08"
-        ixz="-9.649E-07"
-        iyy="0.0072632"
-        iyz="8.7687E-05"
-        izz="0.015199"
-        color = 'orange' />
-<revolute_joint name="R_Knee" type="revolute"
-      origin_xyz="0 -0.28 0"
-      origin_rpy="3.1416 0 3.1416"
-        parent="R_Knee_Upper" child="R_Knee_Lower"
-        limit_e="${Knee_max_effort}" limit_l="${lower_angle}" limit_u="${upper_angle}" limit_v="${angular_velocity}"
-        axis_xyz="1 0 0" />
-<link_stl_box name="R_FootR"
-        origin_xyz="-0.00069157 0.029306 0.012871"
+        parent="R_FootR" child="R_FootS"
+        limit_e="${FootS_max_effort}" limit_l="-0.297" limit_u="0.297" limit_v="${angular_velocity_foot}"
+        joint_damping ="${leg_joint_damping}"  joint_friction ="${leg_joint_friction}"
+        axis_xyz="0 0 1"  />
+<!--Left leg -->
+<revolute_joint name="L_HipR" type="revolute"
+        origin_xyz="0.088 -0.027645 0"
+        origin_rpy="1.5708 0 0"
+        parent="base_link" child="L_HipR"
+        limit_e="${HipR_max_effort}" limit_l="-0.175" limit_u="0.175" limit_v="${angular_velocity_hip}"
+        joint_damping ="${leg_joint_damping}"  joint_friction ="${leg_joint_friction}"
+        axis_xyz="0 1 0"  />
+<revolute_joint name="L_HipS" type="revolute"
+        origin_xyz="0 -0.102 0"
         origin_rpy="0 0 0"
-        box_size = "0.001 0.001 0.001"
-        mass="1.1565"
-        ixx="0.00063348"
-        ixy="-6.7285E-07"
-        ixz="-4.078E-08"
-        iyy="0.00057147"
-        iyz="-3.7116E-06"
-        izz="0.0003019"
-        color = 'orange' />
-<revolute_joint name="R_FootF" type="revolute"
-      origin_xyz="0 -0.27682 0.010063"
-      origin_rpy="3.1053 -0.00039391 -0.010836"
-        parent="R_Knee_Lower" child="R_FootR"
-        limit_e="${FootF_max_effort}" limit_l="${lower_angle}" limit_u="${upper_angle}" limit_v="${angular_velocity}"
-        axis_xyz="0.99994 -0.010843 0"   />
-<link_stl name="R_FootS"
-        origin_xyz="-6.0221E-05 0.080294 -0.056863"
+        parent="L_HipR" child="L_HipS"
+        limit_e="${HipS_max_effort}" limit_l="-0.314" limit_u="0.192" limit_v="${angular_velocity_hip}"
+        joint_damping ="${leg_joint_damping}"  joint_friction ="${leg_joint_friction}"
+        axis_xyz="0 0 1"  />
+<revolute_joint name="L_HipF" type="revolute"
+        origin_xyz="0 0 0"
         origin_rpy="0 0 0"
-        mass="11.269"
-        ixx="0.02985"
-        ixy="-1.1479E-05"
-        ixz="7.8243E-06"
-        iyy="0.03455"
-        iyz="0.00043103"
-        izz="0.0088348"
-        color = 'orange' />
-<revolute_joint name="R_FootS" type="revolute"
-      origin_xyz="-0.00032467 0.030005 0"
-      origin_rpy="0 0 0"
-        parent="R_FootR" child="R_FootS"
-        limit_e="${FootS_max_effort}" limit_l="${lower_angle}" limit_u="${upper_angle}" limit_v="${angular_velocity}"
-        axis_xyz="0 0 1"  />
-<!-- Left Leg -->
-<link_stl_box name="L_HipR"
-        origin_xyz="-0.00070201 -0.027248 -0.022799"
-        origin_rpy="0 0 0"
-        box_size = "0.001 0.001 0.001"
-        mass="2.388"
-        ixx="0.00324"
-        ixy="-1.8675E-05"
-        ixz="4.6222E-05"
-        iyy="0.003218"
-        iyz="7.5574E-06"
-        izz="0.0025543"
-        color = 'orange' />
-<revolute_joint name="L_HipR" type="revolute"
-      origin_xyz="0.088 -0.027645 0"
-      origin_rpy="1.5708 0 0"
-        parent="base_link" child="L_HipR"
-        limit_e="${HipR_max_effort}" limit_l="${lower_angle}" limit_u="${upper_angle}" limit_v="${angular_velocity}"
-        axis_xyz="0 1 0"  />
-<link_stl_box name="L_HipS"
-        origin_xyz="0.0033351 0.00011632 -0.025364"
-        origin_rpy="0 0 0"
-        box_size = "0.001 0.001 0.001"
-        mass="6.15"
-        ixx="0.005105"
-        ixy="1.2895E-05"
-        ixz="1.554E-07"
-        iyy="0.0048687"
-        iyz="1.0129E-05"
-        izz="0.006262"
-        color = 'orange' />
-<revolute_joint name="L_HipS" type="revolute"
-      origin_xyz="0 -0.102 0"
-      origin_rpy="0 0 0"
-        parent="L_HipR" child="L_HipS"
-        limit_e="${HipS_max_effort}" limit_l="${lower_angle}" limit_u="${upper_angle}" limit_v="${angular_velocity}"
-        axis_xyz="0 0 1"  />
-<link_stl_box name="L_Knee_upper"
-        origin_xyz="0.018739 -0.22354 0.0087895"
-        origin_rpy="0 0 0"
-        box_size = "0.001 0.001 0.001"
-        mass="16.528"
-        ixx="0.048222"
-        ixy="4.2459E-06"
-        ixz="6.2369E-05"
-        iyy="0.015119"
-        iyz="0.002184"
-        izz="0.039943"
-        color = 'orange' />
-<revolute_joint name="L_HipF" type="revolute"
-      origin_xyz="0 0 0"
-      origin_rpy="0 0 0"
         parent="L_HipS" child="L_Knee_upper"
-        limit_e="${HipF_max_effort}" limit_l="${lower_angle}" limit_u="${upper_angle}" limit_v="${angular_velocity}"
+        limit_e="${HipF_max_effort}" limit_l="-1.047" limit_u="0.698" limit_v="${angular_velocity_hip}"
+        joint_damping ="${leg_joint_damping}"  joint_friction ="${leg_joint_friction}"
         axis_xyz="1 0 0"  />
-<link_stl_box name="L_Knee_Lower"
-        origin_xyz="0.011812 -0.16731 -0.0034716"
-        origin_rpy="0 0 0"
-        box_size = "0.001 0.001 0.001"
-        mass="10.498"
-        ixx="0.021077"
-        ixy="-1.0082E-06"
-        ixz="-1.8986E-06"
-        iyy="0.007636"
-        iyz="-0.00016695"
-        izz="0.01553"
-        color = 'orange' />
 <revolute_joint name="L_Knee" type="revolute"
       origin_xyz="0 -0.28 0"
-      origin_rpy="-0.036336 0 0"
+      origin_rpy="0 0 0"
         parent="L_Knee_upper" child="L_Knee_Lower"
-        limit_e="${Knee_max_effort}" limit_l="${lower_angle}" limit_u="${upper_angle}" limit_v="${angular_velocity}"
+        limit_e="${Knee_max_effort}" limit_l="-0.087" limit_u="1.571" limit_v="${angular_velocity_knee}"
+        joint_damping ="${leg_joint_damping}"  joint_friction ="${leg_joint_friction}"
         axis_xyz="1 0 0"  />
-<link_stl_box name="L_FootR"
-        origin_xyz="0.00060836 0.029292 0.012871"
-        origin_rpy="0 0 0"
-        box_size = "0.001 0.001 0.001"
-        mass="1.1565"
-        ixx="0.00063348"
-        ixy="-6.7285E-07"
-        ixz="-4.078E-08"
-        iyy="0.00057147"
-        iyz="-3.7116E-06"
-        izz="0.0003019"
-        color = 'orange' />
 <revolute_joint name="L_FootF" type="revolute"
       origin_xyz="0 -0.277 0"
-      origin_rpy="3.1416 0 -0.010843"
+      origin_rpy="3.1416 0 0"
         parent="L_Knee_Lower" child="L_FootR"
-        limit_e="${FootF_max_effort}" limit_l="${lower_angle}" limit_u="${upper_angle}" limit_v="${angular_velocity}"
-        axis_xyz="0.99994 -0.010843 0"  />
-<link_stl name="L_FootS"
-        origin_xyz="-6.0221E-05 0.080294 -0.056863"
-        origin_rpy="0 0 0"
-        mass="11.269"
-        ixx="0.02985"
-        ixy="-1.1479E-05"
-        ixz="7.8243E-06"
-        iyy="0.03455"
-        iyz="0.00043103"
-        izz="0.0088348"
-        color = 'orange' />
+        limit_e="${FootF_max_effort}" limit_l="-1.047" limit_u="0.559" limit_v="${angular_velocity_foot}"
+        joint_damping ="${leg_joint_damping}"  joint_friction ="${leg_joint_friction}"
+        axis_xyz="1 0 0"  />
 <revolute_joint name="L_FootS" type="revolute"
-      origin_xyz="0.00097526 0.029991 0"
+      origin_xyz="0.0 0.030 0"
       origin_rpy="0 0 0"
         parent="L_FootR" child="L_FootS"
-        limit_e="${FootS_max_effort}" limit_l="${lower_angle}" limit_u="${upper_angle}" limit_v="${angular_velocity}"
+        limit_e="${FootS_max_effort}" limit_l="-0.297" limit_u="0.297" limit_v="${angular_velocity_foot}"
+        joint_damping ="${leg_joint_damping}"  joint_friction ="${leg_joint_friction}"
         axis_xyz="0 0 1"  />
+<!--
+<gazebo reference="L_FootS">
+<kp>${ground_kp}</kp>
+<kd>${ground_kd}</kd>
+<mu1>${ground_mu1}</mu1>
+<mu2>${ground_mu2}</mu2>
+<fdir1>1 0 0</fdir1>
+<maxVel>1.0</maxVel>
+<minDepth>0.00</minDepth>
+<maxContacts>4</maxContacts>
+</gazebo>
+<gazebo reference="R_FootS">
+<kp>${ground_kp}</kp>
+<kd>${ground_kd}</kd>
+<mu1>${ground_mu1}</mu1>
+<mu2>${ground_mu2}</mu2>
+<fdir1>1 0 0</fdir1>
+<maxVel>1.0</maxVel>
+<minDepth>0.00</minDepth>
+<maxContacts>4</maxContacts>
+</gazebo> -->
 </robot>

File: src/a600_description/xacro/links_joints_macro.xacro (robot description, xacro)
@@ -2,10 +2,10 @@
 <robot xmlns:xacro="http://www.ros.org/wiki/xacro">
   <!-- Link description -->
-  <xacro:macro name="link_stl" params="name color origin_xyz origin_rpy mass ixx ixy ixz iyy iyz izz">
+  <xacro:macro name="link_stl" params="name color origin_xyz origin_rpy mass ixx iyy izz">
     <link name="${name}">
       <inertial>
         <mass value="${mass}" />
         <origin rpy="${origin_rpy}" xyz="${origin_xyz}" />
-        <inertia ixx="${ixx}" ixy="${ixy}" ixz="${ixz}" iyy="${iyy}" iyz="${iyz}" izz="${izz}" />
+        <inertia ixx="${ixx}" ixy="0.0" ixz="0.0" iyy="${iyy}" iyz="0.0" izz="${izz}" />
       </inertial>
       <collision>
@@ -24,14 +24,14 @@
     </link>
   </xacro:macro>
-   <!-- Link description -->
-  <xacro:macro name="link_stl_box" params="name color origin_xyz origin_rpy box_size mass ixx ixy ixz iyy iyz izz">
+   <!-- Link description with colision box-->
+  <xacro:macro name="link_stl_box" params="name color origin_xyz origin_rpy collision_rpy collision_xyz box_size mass ixx iyy izz">
     <link name="${name}">
       <inertial>
         <mass value="${mass}" />
         <origin rpy="${origin_rpy}" xyz="${origin_xyz}" />
-        <inertia ixx="${ixx}" ixy="${ixy}" ixz="${ixz}" iyy="${iyy}" iyz="${iyz}" izz="${izz}" />
+        <inertia ixx="${ixx}" ixy="0.0" ixz="0.0" iyy="${iyy}" iyz="0.0" izz="${izz}" />
       </inertial>
       <collision>
-        <origin rpy="0 0 0" xyz="0 0 0" />
+        <origin rpy="${collision_rpy}" xyz="${collision_xyz}" />
           <geometry>
           <box size="${box_size}"/>
@@ -40,6 +40,8 @@
       </collision>
       <visual>
+        <!-- <origin rpy="${collision_rpy}" xyz="${collision_xyz}" /> -->
         <origin rpy="0 0 0" xyz="0 0 0" />
         <geometry>
+            <!-- <box size="${box_size}"/> -->
             <mesh filename="package://a600_description/meshes_light/${name}.STL" />
         </geometry>
@@ -49,6 +51,6 @@
   </xacro:macro>
  <!-- Joint description -->
-  <xacro:macro name="revolute_joint" params="name type axis_xyz origin_rpy origin_xyz parent child limit_e limit_l limit_u limit_v">
-    <joint name="${name}" type="${type}">
+  <xacro:macro name="revolute_joint" params="name type axis_xyz origin_rpy origin_xyz parent child limit_e limit_l limit_u limit_v joint_damping joint_friction ">
+    <joint name="${name}" type="${type}" >
       <axis xyz="${axis_xyz}" />
       <limit effort="${limit_e}" lower="${limit_l}" upper="${limit_u}" velocity="${limit_v}" />
@@ -56,4 +58,5 @@
       <parent link="${parent}" />
       <child link="${child}" />
+      <dynamics damping="${joint_damping}" friction="${joint_friction}" />
     </joint>
     <!-- transmission -->

Commit message: fixed joint

File: src/a600_description/xacro/a600_description_box_colision.xacro (robot description, xacro)
@@ -29,5 +29,5 @@
 <xacro:property name="leg_joint_friction"  value="10" />
 <!-- Joint decription-->
-<revolute_joint name="R_HipR" type="revolute"
+<revolute_joint name="R_HipR"
         origin_rpy="1.5708 0 0"
         origin_xyz="-0.088 -0.027645 0"
@@ -36,5 +36,5 @@
         joint_damping ="${leg_joint_damping}"  joint_friction ="${leg_joint_friction}"
         axis_xyz="0 1 0" />
-<revolute_joint name="R_HipS" type="revolute"
+<fixed_joint name="R_HipS"
         origin_xyz="0 -0.102 0"
         origin_rpy="3.1416 0 3.1416"
@@ -43,5 +43,5 @@
         joint_damping ="${leg_joint_damping}"  joint_friction ="${leg_joint_friction}"
         axis_xyz="0 0 1" />
-<revolute_joint name="R_HipF" type="revolute"
+<fixed_joint name="R_HipF"
         origin_xyz="0 0 0"
         origin_rpy="0 0 0"
@@ -50,5 +50,5 @@
         joint_damping ="${leg_joint_damping}"  joint_friction ="${leg_joint_friction}"
         axis_xyz="1 0 0" />
-<revolute_joint name="R_Knee" type="revolute"
+<fixed_joint name="R_Knee"
         origin_xyz="0 -0.28 0"
         origin_rpy="3.1416 0 3.1416"
@@ -57,5 +57,5 @@
         joint_damping ="${leg_joint_damping}"  joint_friction ="${leg_joint_friction}"
         axis_xyz="1 0 0" />
-<revolute_joint name="R_FootF" type="revolute"
+<fixed_joint name="R_FootF"
         origin_xyz="0 -0.277 0.0"
         origin_rpy="3.1416 0 0"
@@ -64,5 +64,5 @@
         joint_damping ="${leg_joint_damping}"  joint_friction ="${leg_joint_friction}"
         axis_xyz="1 0 0"   />
-<revolute_joint name="R_FootS" type="revolute"
+<fixed_joint name="R_FootS"
         origin_xyz="0 0.030 0"
         origin_rpy="0 0 0"
@@ -72,5 +72,5 @@
         axis_xyz="0 0 1"  />
 <!--Left leg -->
-<revolute_joint name="L_HipR" type="revolute"
+<fixed_joint name="L_HipR"
         origin_xyz="0.088 -0.027645 0"
         origin_rpy="1.5708 0 0"
@@ -79,5 +79,5 @@
         joint_damping ="${leg_joint_damping}"  joint_friction ="${leg_joint_friction}"
         axis_xyz="0 1 0"  />
-<revolute_joint name="L_HipS" type="revolute"
+<fixed_joint name="L_HipS"
         origin_xyz="0 -0.102 0"
         origin_rpy="0 0 0"
@@ -86,5 +86,5 @@
         joint_damping ="${leg_joint_damping}"  joint_friction ="${leg_joint_friction}"
         axis_xyz="0 0 1"  />
-<revolute_joint name="L_HipF" type="revolute"
+<fixed_joint name="L_HipF"
         origin_xyz="0 0 0"
         origin_rpy="0 0 0"
@@ -93,5 +93,5 @@
         joint_damping ="${leg_joint_damping}"  joint_friction ="${leg_joint_friction}"
         axis_xyz="1 0 0"  />
-<revolute_joint name="L_Knee" type="revolute"
+<fixed_joint name="L_Knee"
       origin_xyz="0 -0.28 0"
       origin_rpy="0 0 0"
@@ -100,5 +100,5 @@
         joint_damping ="${leg_joint_damping}"  joint_friction ="${leg_joint_friction}"
         axis_xyz="1 0 0"  />
-<revolute_joint name="L_FootF" type="revolute"
+<fixed_joint name="L_FootF"
       origin_xyz="0 -0.277 0"
       origin_rpy="3.1416 0 0"
@@ -107,5 +107,5 @@
         joint_damping ="${leg_joint_damping}"  joint_friction ="${leg_joint_friction}"
         axis_xyz="1 0 0"  />
-<revolute_joint name="L_FootS" type="revolute"
+<fixed_joint name="L_FootS"
       origin_xyz="0.0 0.030 0"
       origin_rpy="0 0 0"

File: src/a600_description/xacro/links_joints_macro.xacro (robot description, xacro)
@@ -51,6 +51,6 @@
   </xacro:macro>
  <!-- Joint description -->
-  <xacro:macro name="revolute_joint" params="name type axis_xyz origin_rpy origin_xyz parent child limit_e limit_l limit_u limit_v joint_damping joint_friction ">
-    <joint name="${name}" type="${type}" >
+  <xacro:macro name="revolute_joint" params="name axis_xyz origin_rpy origin_xyz parent child limit_e limit_l limit_u limit_v joint_damping joint_friction ">
+    <joint name="${name}" type="revolute" >
       <axis xyz="${axis_xyz}" />
       <limit effort="${limit_e}" lower="${limit_l}" upper="${limit_u}" velocity="${limit_v}" />
@@ -71,4 +71,15 @@
       </actuator>
     </transmission>
+  </xacro:macro>
+ <!-- Joint description -->
+  <xacro:macro name="fixed_joint" params="name axis_xyz origin_rpy origin_xyz parent child limit_e limit_l limit_u limit_v joint_damping joint_friction ">
+    <joint name="${name}" type="fixed" >
+      <axis xyz="${axis_xyz}" />
+      <limit effort="${limit_e}" lower="${limit_l}" upper="${limit_u}" velocity="${limit_v}" />
+      <origin rpy="${origin_rpy}" xyz="${origin_xyz}" />
+      <parent link="${parent}" />
+      <child link="${child}" />
+      <dynamics damping="${joint_damping}" friction="${joint_friction}" />
+    </joint>
   </xacro:macro>
 <!-- Color -->
