Commit message: inverse kine done

File: src/a600_description/xacro/links_joints_macro.xacro (robot description, xacro)
@@ -36,5 +36,5 @@
           <geometry>
           <box size="${box_size}"/>
-            <!-- <mesh filename="package://a600_description/meshes/${name}.STL" /> -->
+            <!-- <mesh filename="package://a600_description/meshes_light/${name}.STL" /> -->
           </geometry>
       </collision>
